File: yaacwk.sch (KiCad schematic (older format))
At the start: 71 parts, among them IC1 ATMEGA644P-P, IC2 TLP627-2, J1 EXT_PWR, J2 AUDIO_IN, J3 TX_PTT, J4 TX_KEY, J5 PADDLES, J6 TTL_SERIAL, J7 HEADER_6, J8 HEADER_11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

Commit message: Yaacwk v1.2 with gerber
Parts:
- removed C13, C15: 220nF, Capacitors_ThroughHole:C_Disc_D7.5_P5, symbol C
- removed J8: HEADER_11, Pin_Headers:Pin_Header_Straight_1x11_Pitch2.54mm, symbol HEADER_11
- added C13, C15: 22uF, Capacitors_THT:CP_Radial_D5.0mm_P2.50mm, symbol yaacwk-rescue:CP1
- added J10, J11, J12: HEADER_9, Pin_Headers:Pin_Header_Straight_1x09_Pitch2.54mm, symbol w_connectors:HEADER_9
- added J8: HEADER_8x2, Pin_Headers:Pin_Header_Straight_2x08_Pitch2.54mm, symbol w_connectors:HEADER_8x2
- BZ1: symbol buzzer -> w_device:buzzer
- C1: footprint Capacitors_ThroughHole:C_Disc_D7.5_P5 -> Capacitors_THT:C_Disc_D3.0mm_W1.6mm_P2.50mm; symbol C-RESCUE-yaacwk -> yaacwk-rescue:C
- C10, C11, C2, C3, C4, C5: footprint Capacitors_ThroughHole:C_Disc_D7.5_P5 -> Capacitors_THT:C_Disc_D3.0mm_W1.6mm_P2.50mm; symbol C -> yaacwk-rescue:C
- C12: footprint Capacitors_ThroughHole:C_Disc_D7.5_P5 -> Capacitors_THT:C_Disc_D3.8mm_W2.6mm_P2.50mm; symbol C -> yaacwk-rescue:C
- C14, C16: symbol CP1 -> yaacwk-rescue:CP1
- C17, C18, C19, C6, C7, C8, C9: footprint Capacitors_ThroughHole:C_Disc_D7.5_P5 -> Capacitors_THT:C_Disc_D3.4mm_W2.1mm_P2.50mm; symbol C -> Device:C
- D1, D2, D3: symbol LED -> yaacwk-rescue:LED
- D4: footprint LEDs:LED_D3.0mm -> LEDs:LED_D4.0mm; symbol LED -> yaacwk-rescue:LED
- D5, D6: symbol D_ALT -> yaacwk-rescue:D_ALT
- DS1: symbol LCD16X2 -> display:LCD16X2
- IC1: symbol ATMEGA644P-P -> yaacwk-rescue:ATMEGA644P-P
- IC2: symbol TLP627-2 -> yaacwk-rescue:TLP627-2
- J1, J9: symbol HEADER_3 -> w_connectors:HEADER_3
- J2: symbol PJ320A_3.5mm_4_conductors_audio_plug -> PJ320A:PJ320A_3.5mm_4_conductors_audio_plug
- J3, J4: symbol CONN_01X02 -> yaacwk-rescue:CONN_01X02
- J5: symbol CONN_01X03 -> yaacwk-rescue:CONN_01X03
- J6, J7: symbol HEADER_6 -> w_connectors:HEADER_6
- L1, L2: symbol INDUCTOR -> w_device:INDUCTOR
- LCDPot2: symbol POT -> yaacwk-rescue:POT
- PS2CONN1: symbol Mini-DIN_6pins_ver4 -> custom_kicad_symbols:Mini-DIN_6pins_ver4
- R1, R12, R13, R14, R15, R16, R2, R3, R4, R5, R9: symbol R -> yaacwk-rescue:R
- R10, R11: symbol R-RESCUE-yaacwk -> yaacwk-rescue:R-RESCUE-yaacwk
- R6, R7, R8: value 470 Ohm -> 1kOhm; symbol R -> yaacwk-rescue:R
- SW1, SW2, SW3, SW4, SW5, SW7, SW8, SW9: footprint Pin_Headers:Pin_Header_Straight_1x02_Pitch2.54mm -> Buttons_Switches_THT:SW_TH_Tactile_Omron_B3F-10xx; symbol SW_PUSH -> w_device:SW_PUSH
- SW6: symbol SW_PUSH -> w_device:SW_PUSH
- SpeedPot1: footprint Potentiometers:Potentiometer_Alps_RK097_Single_Vertical -> Potentiometers:Potentiometer_Piher_T16H_Single_Vertical; symbol POT -> yaacwk-rescue:POT
- U1, U2: symbol LM7805 -> yaacwk-rescue:LM7805
- Y1: symbol Crystal -> yaacwk-rescue:Crystal
Connections:
- wire segments 249 -> 421
- no-connect marks 11 -> 10
Other:
- moved on the sheet: C17, C18, C19, C6, C7, C8, C9, D1, D2, D3, R1, R14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

Commit message: Yaacwk v1.3 with gerber and current WIP
Parts:
- removed J1: EXT_PWR, Connectors:BARREL_JACK, symbol w_connectors:HEADER_3
- removed J3: TX_PTT, Pin_Headers:Pin_Header_Straight_1x02_Pitch2.54mm, symbol yaacwk-rescue:CONN_01X02
- removed J4: TX_KEY, Pin_Headers:Pin_Header_Straight_1x02_Pitch2.54mm, symbol yaacwk-rescue:CONN_01X02
- removed J5: PADDLES, Pin_Headers:Pin_Header_Straight_1x03_Pitch2.54mm, symbol yaacwk-rescue:CONN_01X03
- added C20: 0.47uF, Capacitors_THT:CP_Radial_D5.0mm_P2.50mm, symbol Device:CP1
- added D7: D_ALT, Diodes_THT:D_A-405_P7.62mm_Horizontal, symbol yaacwk-rescue:D_ALT
- added J1: EXT_PWR, Connectors:BARREL_JACK, symbol Connector:Barrel_Jack_Switch
- added J3: TX_PTT, PJRAN1X1U03AUX:PJRAN1X1U03AUX, symbol PJRAN1X1U03AUX:PJRAN1X1U03AUX
- added J4: TX_KEY, PJRAN1X1U03AUX:PJRAN1X1U03AUX, symbol PJRAN1X1U03AUX:PJRAN1X1U03AUX
- added J5: PADDLES, PJ320A:PJ320A_3.5mm_4_conductors_audio_plug, symbol PJ320A:PJ320A_3.5mm_4_conductors_audio_plug
- added R17: 10kOhm, Resistors_THT:R_Axial_DIN0207_L6.3mm_D2.5mm_P7.62mm_Horizontal, symbol Device:R
- J8: value HEADER_8x2 -> HEADER_9x2; footprint Pin_Headers:Pin_Header_Straight_2x08_Pitch2.54mm -> Pin_Headers:Pin_Header_Straight_2x09_Pitch2.54mm; symbol w_connectors:HEADER_8x2 -> w_connectors:HEADER_9x2
- J9: footprint Pin_Headers:Pin_Header_Straight_1x03_Pitch2.54mm -> Pin_Headers:Pin_Header_Straight_2x03_Pitch2.54mm; symbol w_connectors:HEADER_3 -> w_connectors:HEADER_3x2
- SW1, SW2, SW3, SW4, SW5, SW7, SW8, SW9: value SW_PUSH -> SW_SPDT; symbol w_device:SW_PUSH -> w_device:SW_SPDT
- SW6: value SW_PUSH -> SW_SPDT; footprint Pin_Headers:Pin_Header_Straight_1x02_Pitch2.54mm -> Buttons_Switches_THT:SW_TH_Tactile_Omron_B3F-10xx; symbol w_device:SW_PUSH -> w_device:SW_SPDT
- U2: value LM2937 -> LM317
Connections:
- net GND: now also J8.18, J1.2, J1.3, J5.5 (GND)
- net at DS1.15 (LED+), DS1.2 (VDD), IC1.10 (VCC)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: now also J9.3, R17.1; no longer C16.1, J9.2, U2.VI
- net at C4.2, C5.2, IC2.5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: now also J3.1 (SLEEVE), J4.1 (SLEEVE)
- net at C5.1, IC2.6: now also J4.2 (TIP), J4.3 (SHUNT)
- net at C4.1, IC2.8: now also J3.2 (TIP), J3.3 (SHUNT)
- net at C2.1, IC1.27 ((PCINT22/TDI)PC5): now also J5.4 (R)
- net at C3.1, IC1.28 ((PCINT23/TOSC1)PC6): now also J5.3 (L)
- net at C8.2, J10.4, J11.4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: now also SW4.3 (NO); no longer SW4.2
- net at C9.2, J10.5, J11.5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: now also SW5.3 (NO); no longer SW5.2
- net at C7.2, J10.3, J11.3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: now also SW3.3 (NO); no longer SW3.2
- net at C6.2, J10.2, J11.2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: now also SW2.3 (NO); no longer SW2.2
- net at IC1.39 ((PCINT1/ADC1)PA1), J10.1, J11.1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: now also SW1.3 (NO); no longer SW1.2
- net at IC1.9 (~RESET): now also J8.17, SW6.3 (NO), C20.2, R17.2; no longer SW6.2
- net at C12.1, J2.3 (L), J2.4 (R): no longer J2.2 (MIC)
- net at D6.2 (A): now also J1.1
- net at C14.1, D6.1 (K), U1.VI: now also C16.1, U2.VI
- net at J6.5: now also C20.1
- net at J6.6: now also D7.2 (A)
- net at D5.1 (K): now also J9.5; no longer J9.3
- net at C17.2, J10.6, J11.6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: now also SW7.3 (NO); no longer SW7.2
- net at C18.2, J10.7, J11.7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: now also SW8.3 (NO); no longer SW8.2
- net at C19.2, J10.8, J11.8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: now also SW9.3 (NO); no longer SW9.2
- net at C15.1, U2.VO: now also J9.2; no longer J8.1, J8.2
- new net: J8.1, J8.2, J9.4
- new net: D7.1 (K), J9.6
Other:
- moved on the sheet: BZ1, C1, C10, C11, C12, C13, C14, C15, C16, C17, C18, C19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
